Commit message: fix more names

File: hungryToaster_description/urdf/hungryToaster_description.urdf (robot description, URDF)
Before this commit: robot hungry-toaster, 2 links, 1 joints
Links:
- link base_link: geometry visual mesh filename=package://hungryToaster_description/meshes/hungry-toaster-m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
