Commit message: fix urdf and conventions

File: hungry_toaster_description/urdf/hungry_toaster_description.urdf (robot description, URDF)
Before this commit: robot hungryToaster, 2 links, 1 joints
Links:
- link base_link: geometry visual mesh filename=package://hungry_toaster_description/meshes/hungry_toaster_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
