Commit message: turn robot around

File: hungry_toaster/urdf/hungry_toaster_description.urdf (robot description, URDF)
Before this commit: robot hungry_toaster, 2 links, 1 joints
Joints:
- joint base_link_to_laser: origin xyz=0.3048 0.254 0.6096 rpy=0 0 -1.57 -> xyz=-0.3048 -0.254 0.6096 rpy=0 0 1.57

Commit message: it works but it disables the map?

File: hungry_toaster/urdf/hungry_toaster_description.urdf (robot description, URDF)
Before this commit: robot hungry_toaster, 2 links, 1 joints
Links:
- link base_link: geometry visual mesh filename=package://hungry_toaster/meshes/hungry_toaster_meters.dae

Commit message: Add limelight link and limelight geometry

File: hungry_toaster/urdf/hungry_toaster_description.urdf (robot description, URDF)
Before this commit: robot hungry_toaster, 2 links, 1 joints
Links:
- added link limelight; visual box size=0.0254 0.09779 0.05715
Joints:
- added joint base_link_to_limelight: type fixed, parent base_link, child limelight, origin xyz=0.0 0.0 0.0 rpy=0 0 0

Commit message: Fixed bugs (still need to fix inversion) thanks mike!

File: hungry_toaster/urdf/hungry_toaster_description.urdf (robot description, URDF)
Before this commit: robot hungry_toaster, 3 links, 2 joints
Joints:
- joint base_link_to_limelight: origin xyz=0.0 0.0 0.0 rpy=0 0 0 -> xyz=0.5 -0.3 0.1 rpy=0 -0.1 0
