Commit message: Add ML camera source to urdf

File: unnamed_toaster/unnamed_toaster/urdf/unnamed_toaster_description.urdf (robot description, URDF)
Before this commit: robot unnamed, 3 links, 2 joints
Links:
- added link ml_link; visual box size=0.0254 0.09779 0.05715
Joints:
- added joint base_link_to_ml_link: type fixed, parent base_link, child ml_link, origin xyz=0 0 0 rpy=0 0 0

Commit message: Update URDF to include turret

File: unnamed_toaster/unnamed_toaster/urdf/unnamed_toaster_description.urdf (robot description, URDF)
Before this commit: robot unnamed, 3 links, 2 joints
Links:
- added link turret; visual cylinder length=0.3 radius=0.55
Joints:
- removed joint base_link_to_limelight
- added joint base_link_to_turret: type revolute, parent base_link, child turret, origin xyz=0.0 0.0 0.0 rpy=0 0 0, axis 0 0 1, limit lower=-6.0 upper=6.0 effort=1000.0 velocity=0.5
- added joint turret_to_limelight: type fixed, parent turret, child limelight, origin xyz=0.5 -0.3 0.1 rpy=0 -0.1 0

Commit message: Replace robot frame

File: unnamed_toaster/unnamed_toaster/urdf/unnamed_toaster_description.urdf (robot description, URDF)
Before this commit: robot unnamed, 3 links, 2 joints
Links:
- link base_link: geometry visual mesh filename=package://unnamed_toaster/meshes/unnamed_toaster_frame.stl

Commit message: Add new turret meshes

File: unnamed_toaster/unnamed_toaster/urdf/unnamed_toaster_description.urdf (robot description, URDF)
Before this commit: robot unnamed, 4 links, 3 joints
Links:
- link base_link: geometry visual mesh filename=package://unnamed_toaster/meshes/unnamed_toaster_meters.stl
- link turret: geometry visual mesh filename=package://unnamed_toaster/meshes/unnamed_toaster_turret.stl

Commit message: fix the orientations

File: unnamed_toaster/unnamed_toaster/urdf/unnamed_toaster_description.urdf (robot description, URDF)
Before this commit: robot unnamed, 4 links, 3 joints
Joints:
- removed joint base_link_to_turret
- added joint turret_joint: type revolute, parent base_link, child turret, origin xyz=-0.0922782 0.0 0.263525 rpy=0.0 0.0 0.0, axis 0 0 1, limit lower=-6.0 upper=6.0 effort=1000.0 velocity=0.5
- joint base_link_to_laser: origin xyz=-0.3048 -0.254 0.6096 rpy=0 0 1.57 -> xyz=-0.193675 0.09525 0.2 rpy=0 0 1.57
- joint turret_to_limelight: origin xyz=0.5 -0.3 0.1 rpy=0 -0.1 0 -> xyz=0.0 0.2428875 0.4318 rpy=0.0 0.0 0.0

Commit message: set laser orientation

File: unnamed_toaster/unnamed_toaster/urdf/unnamed_toaster_description.urdf (robot description, URDF)
Before this commit: robot unnamed, 4 links, 3 joints
Joints:
- joint base_link_to_laser: origin xyz=-0.193675 0.09525 0.2 rpy=0 0 1.57 -> xyz=-0.193675 0.09525 0.2 rpy=3.14 0 3.14
